File: input.kicad_sch (KiCad schematic)
At the start: 31 parts

Commit message: routing progress towards v001
Parts:
- BTN3, BTN4, ID3, ID4, R3, R4: now left out of the parts list
Other:
- note added: "not on v0"
Changed lines of the file:
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@@
     (stroke (width 0) (type default))
+  )
+  (rectangle (start 36.83 57.15) (end 66.04 74.93)
+    (stroke (width 0) (type default))
+    (fill (type none))
+  )
+  (text "not on v0" (at 25.4 73.66 0)
+    (effects (font (size 1.27 1.27)) (justify left bottom))
   )
   (hierarchical_label "INT" (shape output) (at 74.93 34.29 0) (fields_autoplaced)
@@
   )
   (symbol (lib_id "Device:D_Schottky") (at 62.23 59.69 180) (unit 1)
-    (in_bom yes) (on_board yes) (dnp no)
+    (in_bom no) (on_board no) (dnp no)
     (property "Reference" "ID3" (at 58.42 58.42 0)
       (effects (font (size 1.27 1.27)))
@@
   )
   (symbol (lib_id "Switch:SW_Push") (at 50.8 62.23 0) (unit 1)
-    (in_bom yes) (on_board yes) (dnp no)
+    (in_bom no) (on_board no) (dnp no)
     (property "Reference" "BTN3" (at 53.34 59.69 0)
       (effects (font (size 1.27 1.27)))
@@
   )
   (symbol (lib_id "Device:R") (at 62.23 64.77 90) (unit 1)
-    (in_bom yes) (on_board yes) (dnp no)
+    (in_bom no) (on_board no) (dnp no)
     (property "Reference" "R3" (at 69.85 64.77 90)
       (effects (font (size 1.27 1.27)))
@@
   )
   (symbol (lib_id "Switch:SW_Push") (at 50.8 71.12 0) (unit 1)
-    (in_bom yes) (on_board yes) (dnp no)
+    (in_bom no) (on_board no) (dnp no)
     (property "Reference" "BTN4" (at 53.34 68.58 0)
       (effects (font (size 1.27 1.27)))
@@
   )
   (symbol (lib_id "Device:D_Schottky") (at 62.23 68.58 180) (unit 1)
-    (in_bom yes) (on_board yes) (dnp no)
+    (in_bom no) (on_board no) (dnp no)
     (property "Reference" "ID4" (at 58.42 67.31 0)
       (effects (font (size 1.27 1.27)))
@@
   )
   (symbol (lib_id "Device:R") (at 62.23 73.66 90) (unit 1)
-    (in_bom yes) (on_board yes) (dnp no)
+    (in_bom no) (on_board no) (dnp no)
     (property "Reference" "R4" (at 69.85 73.66 90)
       (effects (font (size 1.27 1.27)))
