File: kontakcount.kicad_sch (KiCad schematic)
At the start: 15 parts

Commit message: routing progress towards v001
Parts:
- added H1, H2, H3, H4: MountingHole_Pad, MountingHole:MountingHole_3.2mm_M3_DIN965_Pad, symbol Mechanical:MountingHole_Pad
- added R23: 0, Resistor_SMD:R_0805_2012Metric_Pad1.20x1.40mm_HandSolder, symbol Device:R
Connections:
- net CLK: now also ESP32-C3.5 (GPIO5)
- net GND: now also H1.1, H2.1, H3.1, H4.1
- net at ESP32-C3.7 (GPIO7), LORA1.3 (MOSI): now also CHSEL1.14 (SER)
- net at ESP32-C3.20 (GPIO20): now also R23.1; no longer RGB1.2 (DIN)
- new net: R23.2, RGB1.2 (DIN)
