File: power.kicad_sch (KiCad schematic)
At the start: 9 parts

Commit message: routing progress towards v001
Parts:
- added SWPWR1: SW_SPDT, xandy1:POWERSWITCH SLIDE THT, symbol Switch:SW_SPDT
- L1: footprint Inductor_SMD:L_1210_3225Metric_Pad1.42x2.65mm_HandSolder -> Inductor_SMD:L_12x12mm_H6mm
Connections:
- net VBATT: now also BUCK1.1 (VIN), Cpwr1.1, Cpwr2.1, Cpwr3.1, Dpwr2.1 (K); no longer BAT1.2 (Pin_2), Dpwr2.2 (A)
- new net: BAT1.2 (Pin_2), SWPWR1.2 (B)
- new net: Dpwr2.2 (A), SWPWR1.1 (A)
- no-connect marks 0 -> 1
Changed lines of the file:
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@@
   (junction (at 121.92 76.2) (diameter 0) (color 0 0 0 0)
   )
+  (junction (at 85.09 57.15) (diameter 0) (color 0 0 0 0)
+  )
   (junction (at 81.28 71.12) (diameter 0) (color 0 0 0 0)
   )
-  (junction (at 73.66 71.12) (diameter 0) (color 0 0 0 0)
-  )
-  (junction (at 58.42 71.12) (diameter 0) (color 0 0 0 0)
-  )
   (junction (at 81.28 82.55) (diameter 0) (color 0 0 0 0)
   )
@@
   (junction (at 106.68 82.55) (diameter 0) (color 0 0 0 0)
   )
+  (junction (at 77.47 71.12) (diameter 0) (color 0 0 0 0)
+  )
+  (no_connect (at 68.58 53.34))
   (wire (pts (xy 133.35 68.58) (xy 133.35 76.2))
     (stroke (width 0) (type default))
@@
     (stroke (width 0) (type default))
   )
-  (wire (pts (xy 60.96 62.23) (xy 58.42 62.23))
-    (stroke (width 0) (type default))
-  )
-  (wire (pts (xy 73.66 71.12) (xy 81.28 71.12))
+  (wire (pts (xy 85.09 57.15) (xy 85.09 54.61))
+    (stroke (width 0) (type default))
+  )
+  (wire (pts (xy 73.66 71.12) (xy 77.47 71.12))
     (stroke (width 0) (type default))
   )
@@
     (stroke (width 0) (type default))
   )
-  (wire (pts (xy 58.42 62.23) (xy 58.42 71.12))
+  (wire (pts (xy 58.42 50.8) (xy 58.42 71.12))
+    (stroke (width 0) (type default))
+  )
+  (wire (pts (xy 85.09 63.5) (xy 85.09 57.15))
     (stroke (width 0) (type default))
   )
@@
     (stroke (width 0) (type default))
   )
+  (wire (pts (xy 68.58 48.26) (xy 72.39 48.26))
+    (stroke (width 0) (type default))
+  )
   (wire (pts (xy 57.15 77.47) (xy 57.15 82.55))
     (stroke (width 0) (type default))
@@
     (stroke (width 0) (type default))
   )
-  (wire (pts (xy 68.58 71.12) (xy 73.66 71.12))
-    (stroke (width 0) (type default))
-  )
   (wire (pts (xy 119.38 68.58) (xy 133.35 68.58))
     (stroke (width 0) (type default))
@@
     (stroke (width 0) (type default))
   )
-  (wire (pts (xy 58.42 71.12) (xy 60.96 71.12))
+  (wire (pts (xy 77.47 71.12) (xy 81.28 71.12))
     (stroke (width 0) (type default))
   )
@@
     (stroke (width 0) (type default))
   )
+  (wire (pts (xy 80.01 63.5) (xy 80.01 68.58))
+    (stroke (width 0) (type default))
+  )
   (wire (pts (xy 81.28 71.12) (xy 87.63 71.12))
     (stroke (width 0) (type default))
@@
     (stroke (width 0) (type default))
   )
+  (wire (pts (xy 77.47 68.58) (xy 77.47 71.12))
+    (stroke (width 0) (type default))
+  )
   (wire (pts (xy 121.92 76.2) (xy 125.73 76.2))
     (stroke (width 0) (type default))
@@
     (stroke (width 0) (type default))
   )
-  (hierarchical_label "VBATT" (shape output) (at 60.96 62.23 0) (fields_autoplaced)
+  (wire (pts (xy 80.01 48.26) (xy 80.01 54.61))
+    (stroke (width 0) (type default))
+  )
+  (wire (pts (xy 85.09 54.61) (xy 80.01 54.61))
+    (stroke (width 0) (type default))
+  )
+  (wire (pts (xy 80.01 63.5) (xy 85.09 63.5))
+    (stroke (width 0) (type default))
+  )
+  (wire (pts (xy 85.09 57.15) (xy 88.9 57.15))
+    (stroke (width 0) (type default))
+  )
+  (wire (pts (xy 80.01 68.58) (xy 77.47 68.58))
+    (stroke (width 0) (type default))
+  )
+  (hierarchical_label "VBATT" (shape output) (at 88.9 57.15 0) (fields_autoplaced)
     (effects (font (size 1.27 1.27)) (justify left))
   )
@@
     )
   )
-  (symbol (lib_id "Device:D_Schottky") (at 64.77 71.12 180) (unit 1)
-    (in_bom yes) (on_board yes) (dnp no) (fields_autoplaced)
-    (property "Reference" "Dpwr2" (at 65.0875 67.31 0)
-      (effects (font (size 1.27 1.27)))
-    )
-    (property "Value" "D_Schottky" (at 63.8175 73.66 90)
-      (effects (font (size 1.27 1.27)) (justify left) hide)
-    )
-    (property "Footprint" "Diode_SMD:D_SMA_Handsoldering" (at 64.77 71.12 0)
-      (effects (font (size 1.27 1.27)) hide)
-    )
-    (property "Datasheet" "~" (at 64.77 71.12 0)
-      (effects (font (size 1.27 1.27)) hide)
-    )
-    (pin "2")
-    (pin "1")
-    (instances
-      (project "kontakcount"
-        (path "/7308d770-83e1-4c62-b394-a56b05c31c12/35ebed86-d97c-4c86-bcff-8cd24a60e53a"
-          (reference "Dpwr2") (unit 1)
-        )
-      )
-    )
-  )
   (symbol (lib_id "Device:D_Schottky") (at 121.92 80.01 270) (unit 1)
     (in_bom yes) (on_board yes) (dnp no) (fields_autoplaced)
@@
     )
   )
+  (symbol (lib_id "Switch:SW_SPDT") (at 63.5 50.8 0) (unit 1)
+    (in_bom yes) (on_board yes) (dnp no) (fields_autoplaced)
+    (property "Reference" "SWPWR1" (at 63.5 43.18 0)
+      (effects (font (size 1.27 1.27)))
+    )
+    (property "Value" "SW_SPDT" (at 63.5 45.72 0)
+      (effects (font (size 1.27 1.27)))
+    )
+    (property "Footprint" "xandy1:POWERSWITCH SLIDE THT" (at 63.5 50.8 0)
+      (effects (font (size 1.27 1.27)) hide)
+    )
+    (property "Datasheet" "~" (at 63.5 50.8 0)
+      (effects (font (size 1.27 1.27)) hide)
+    )
+    (pin "1")
+    (pin "2")
+    (pin "3")
+    (instances
+      (project "kontakcount"
+        (path "/7308d770-83e1-4c62-b394-a56b05c31c12/35ebed86-d97c-4c86-bcff-8cd24a60e53a"
+          (reference "SWPWR1") (unit 1)
+        )
+      )
+    )
+  )
+  (symbol (lib_id "Device:D_Schottky") (at 76.2 48.26 180) (unit 1)
+    (in_bom yes) (on_board yes) (dnp no) (fields_autoplaced)
+    (property "Reference" "Dpwr2" (at 76.5175 44.45 0)
+      (effects (font (size 1.27 1.27)))
+    )
+    (property "Value" "D_Schottky" (at 75.2475 50.8 90)
+      (effects (font (size 1.27 1.27)) (justify left) hide)
+    )
+    (property "Footprint" "Diode_SMD:D_SMA_Handsoldering" (at 76.2 48.26 0)
+      (effects (font (size 1.27 1.27)) hide)
+    )
+    (property "Datasheet" "~" (at 76.2 48.26 0)
+      (effects (font (size 1.27 1.27)) hide)
+    )
+    (pin "2")
+    (pin "1")
+    (instances
+      (project "kontakcount"
+        (path "/7308d770-83e1-4c62-b394-a56b05c31c12/35ebed86-d97c-4c86-bcff-8cd24a60e53a"
+          (reference "Dpwr2") (unit 1)
+        )
+      )
+    )
+  )
   (symbol (lib_id "Device:C_Polarized") (at 81.28 74.93 0) (unit 1)
     (in_bom yes) (on_board yes) (dnp no)
@@
       (effects (font (size 1.27 1.27)))
     )
-    (property "Footprint" "Inductor_SMD:L_1210_3225Metric_Pad1.42x2.65mm_HandSolder" (at 129.54 76.2 0)
-      (effects (font (size 1.27 1.27)) hide)
-    )
+    (property "Footprint" "Inductor_SMD:L_12x12mm_H6mm" (at 129.54 76.2 0)
+      (effects (font (size 1.27 1.27)) hide)
+    )
